File: Eagle/Lulu_MCU/Lulu_MCU.brd (EAGLE design)
At the start: 12.4 x 12.4 mm, 3 parts

Commit message: Initial commit from Lucette branche
Parts:
- added U1: (no value), microbuilder:MLF20_4X4MM_0.5MM_ATMEL
Connections:
- new net GND: U1.8, U1.THERMAL
- new net VCC: U1.15
Changed lines of the file:
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@@
 <?xml version="1.0" encoding="utf-8"?>
 <!DOCTYPE eagle SYSTEM "eagle.dtd">
-<eagle version="6.5.0">
+<eagle version="8.4.3">
 <drawing>
 <settings>
 <setting alwaysvectorfont="no"/>
+<setting keepoldvectorfont="yes"/>
 <setting verticaltext="up"/>
 </settings>
@@
 <layer number="59" name="tCarbon" color="7" fill="1" visible="no" active="no"/>
 <layer number="60" name="bCarbon" color="7" fill="1" visible="no" active="no"/>
-<layer number="90" name="Modules" color="5" fill="1" visible="yes" active="yes"/>
+<layer number="90" name="Modules" color="5" fill="1" visible="no" active="no"/>
 <layer number="91" name="Nets" color="2" fill="1" visible="no" active="no"/>
 <layer number="92" name="Busses" color="1" fill="1" visible="no" active="no"/>
@@
 <layer number="230" name="230bmp" color="7" fill="1" visible="yes" active="yes"/>
 <layer number="231" name="231bmp" color="7" fill="1" visible="yes" active="yes"/>
+<layer number="232" name="Eagle3D_PG2" color="7" fill="1" visible="no" active="no"/>
+<layer number="233" name="Eagle3D_PG3" color="7" fill="1" visible="no" active="no"/>
 <layer number="248" name="Housing" color="7" fill="1" visible="yes" active="yes"/>
 <layer number="249" name="Edge" color="7" fill="1" visible="yes" active="yes"/>
@@
 <param name="dpMaxLengthDifference" value="10mm"/>
 <param name="dpGapFactor" value="2.5"/>
-<param name="checkGrid" value="0"/>
 <param name="checkAngle" value="0"/>
 <param name="checkFont" value="1"/>
 <param name="checkRestrict" value="0"/>
+<param name="checkStop" value="0"/>
 <param name="useDiameter" value="13"/>
 <param name="maxErrors" value="50"/>
@@
 <pass name="Default">
 <param name="RoutingGrid" value="50mil"/>
+<param name="AutoGrid" value="1"/>
+<param name="Efforts" value="0"/>
+<param name="TopRouterVariant" value="1"/>
 <param name="tpViaShape" value="round"/>
 <param name="PrefDir.1" value="|"/>
@@
 <element name="JP4" library="LilyPad-Wearables" package="PETAL-SMALL" value="SEWTAP4" x="2.38125" y="6.19125" rot="R270"/>
 <element name="U$1" library="OSRAM" package="OSLON" value="OSRAM_SMT" x="6.50875" y="9.8425"/>
+<element name="U1" library="microbuilder" package="MLF20_4X4MM_0.5MM_ATMEL" value="" x="20.32" y="6.35"/>
 </elements>
 <signals>
@@
 <vertex x="2.19" y="2.1275" curve="-90"/>
 </polygon>
+<contactref element="U1" pad="THERMAL"/>
+<contactref element="U1" pad="8"/>
+<wire x1="20.32" y1="6.35" x2="20.32" y2="4.35" width="0" layer="19" extent="1-1"/>
+</signal>
+<signal name="VCC">
+<contactref element="U1" pad="15"/>
 </signal>
 </signals>
