File: Eagle/Lulu_MCU/Lulu_MCU.sch (EAGLE design)
At the start: 3 parts

Commit message: Initial commit from Lucette branche
Parts:
- added U1: (no value), microbuilder:ATTINY85
Changed lines of the file:
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@@
 <?xml version="1.0" encoding="utf-8"?>
 <!DOCTYPE eagle SYSTEM "eagle.dtd">
-<eagle version="6.5.0">
+<eagle version="8.4.3">
 <drawing>
 <settings>
 <setting alwaysvectorfont="no"/>
+<setting keepoldvectorfont="yes"/>
 <setting verticaltext="up"/>
 </settings>
@@
 <layer number="230" name="230bmp" color="7" fill="1" visible="yes" active="yes"/>
 <layer number="231" name="231bmp" color="7" fill="1" visible="yes" active="yes"/>
+<layer number="232" name="Eagle3D_PG2" color="7" fill="1" visible="no" active="no"/>
+<layer number="233" name="Eagle3D_PG3" color="7" fill="1" visible="no" active="no"/>
 <layer number="248" name="Housing" color="7" fill="1" visible="no" active="yes"/>
 <layer number="249" name="Edge" color="7" fill="1" visible="no" active="yes"/>
@@
 <part name="JP4" library="LilyPad-Wearables" deviceset="SEWTAP" device="4" value="SEWTAP4"/>
 <part name="U$1" library="OSRAM" deviceset="OSRAM_SMT" device=""/>
+<part name="U1" library="microbuilder" deviceset="ATTINY85" device=""/>
 </parts>
 <sheets>
@@
 <instance part="JP4" gate="G$1" x="50.8" y="38.1"/>
 <instance part="U$1" gate="LED" x="35.56" y="38.1"/>
+<instance part="U1" gate="G$1" x="38.1" y="7.62"/>
 </instances>
 <busses>
@@
 </schematic>
 </drawing>
+<compatibility>
+<note version="6.3" minversion="6.2.2" severity="warning">
+Since Version 6.2.2 text objects can contain more than one line,
+which will not be processed correctly with this version.
+</note>
+</compatibility>
 </eagle>
