File: Hardware/kicad_Lulu_star/Lulu_star_212/_autosave-Lulu_star_212.kicad_pcb (KiCad board)
At the start: 2 copper layers, 16.7 x 14.9 mm, 6 parts, among them J1 Conn_01x03_Female, Q1 Q_NMOS_GSD, T1 Q_NPN_BEC

Commit message: PCB in progress
Parts:
- moved Q1 0.25 mm to (128.0, 102.9)
- moved R1 0.25 mm to (125.5, 100.3)
- moved T1 0.25 mm to (124.2, 102.9)
Changed lines of the file:
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@@
       (effects (font (size 1 1) (thickness 0.15)))
     )
+    (fp_poly (pts (xy -0.762 2.54) (xy 0.762 2.54) (xy 0.762 0) (xy -0.762 0)) (layer F.Mask) (width 0.15))
+    (fp_poly (pts (xy -0.762 2.54) (xy 0.762 2.54) (xy 0.762 0) (xy -0.762 0)) (layer F.Cu) (width 0.15))
+    (fp_arc (start 0 2.54) (end -0.762 2.54) (angle -180) (layer F.Cu) (width 0.17))
+    (fp_arc (start 0 0) (end 0.762 0) (angle -180) (layer F.Mask) (width 0.17))
+    (fp_line (start -0.762 2.54) (end -0.762 0) (layer F.Cu) (width 0.17))
+    (fp_line (start 0.762 0) (end 0.762 2.54) (layer F.Mask) (width 0.17))
+    (fp_line (start 0.762 0) (end 0.762 2.54) (layer F.Cu) (width 0.17))
+    (fp_arc (start 0 0) (end 0.762 0) (angle -180) (layer F.Cu) (width 0.17))
+    (fp_arc (start 0 2.54) (end -0.762 2.54) (angle -180) (layer F.Mask) (width 0.17))
+    (fp_line (start -0.762 2.54) (end -0.762 0) (layer F.Mask) (width 0.17))
+    (fp_poly (pts (xy 1.778 2.54) (xy 3.302 2.54) (xy 3.302 0) (xy 1.778 0)) (layer F.Mask) (width 0.15))
+    (fp_poly (pts (xy 1.778 2.54) (xy 3.302 2.54) (xy 3.302 0) (xy 1.778 0)) (layer F.Cu) (width 0.15))
+    (fp_arc (start 2.54 2.54) (end 1.778 2.54) (angle -180) (layer F.Cu) (width 0.17))
+    (fp_arc (start 2.54 0) (end 3.302 0) (angle -180) (layer F.Mask) (width 0.17))
+    (fp_line (start 1.778 2.54) (end 1.778 0) (layer F.Cu) (width 0.17))
+    (fp_line (start 3.302 0) (end 3.302 2.54) (layer F.Mask) (width 0.17))
+    (fp_line (start 3.302 0) (end 3.302 2.54) (layer F.Cu) (width 0.17))
+    (fp_arc (start 2.54 0) (end 3.302 0) (angle -180) (layer F.Cu) (width 0.17))
+    (fp_arc (start 2.54 2.54) (end 1.778 2.54) (angle -180) (layer F.Mask) (width 0.17))
+    (fp_line (start 1.778 2.54) (end 1.778 0) (layer F.Mask) (width 0.17))
+    (fp_poly (pts (xy 4.318 2.54) (xy 5.842 2.54) (xy 5.842 0) (xy 4.318 0)) (layer F.Cu) (width 0.15))
+    (fp_line (start 4.318 2.54) (end 4.318 0) (layer F.Mask) (width 0.17))
+    (fp_arc (start 5.08 2.54) (end 4.318 2.54) (angle -180) (layer F.Mask) (width 0.17))
+    (fp_line (start 5.842 0) (end 5.842 2.54) (layer F.Mask) (width 0.17))
+    (fp_arc (start 5.08 0) (end 5.842 0) (angle -180) (layer F.Mask) (width 0.17))
+    (fp_line (start 4.318 2.54) (end 4.318 0) (layer F.Cu) (width 0.17))
+    (fp_arc (start 5.08 2.54) (end 4.318 2.54) (angle -180) (layer F.Cu) (width 0.17))
+    (fp_line (start 5.842 0) (end 5.842 2.54) (layer F.Cu) (width 0.17))
+    (fp_arc (start 5.08 0) (end 5.842 0) (angle -180) (layer F.Cu) (width 0.17))
     (fp_poly (pts (xy 4.318 2.54) (xy 5.842 2.54) (xy 5.842 0) (xy 4.318 0)) (layer F.Mask) (width 0.15))
-    (fp_arc (start 5.08 0) (end 5.842 0) (angle -180) (layer F.Cu) (width 0.17))
-    (fp_line (start 5.842 0) (end 5.842 2.54) (layer F.Cu) (width 0.17))
-    (fp_arc (start 5.08 2.54) (end 4.318 2.54) (angle -180) (layer F.Cu) (width 0.17))
-    (fp_line (start 4.318 2.54) (end 4.318 0) (layer F.Cu) (width 0.17))
-    (fp_arc (start 5.08 0) (end 5.842 0) (angle -180) (layer F.Mask) (width 0.17))
-    (fp_line (start 5.842 0) (end 5.842 2.54) (layer F.Mask) (width 0.17))
-    (fp_arc (start 5.08 2.54) (end 4.318 2.54) (angle -180) (layer F.Mask) (width 0.17))
-    (fp_line (start 4.318 2.54) (end 4.318 0) (layer F.Mask) (width 0.17))
-    (fp_poly (pts (xy 4.318 2.54) (xy 5.842 2.54) (xy 5.842 0) (xy 4.318 0)) (layer F.Cu) (width 0.15))
+    (pad 1 thru_hole circle (at 0 2.54) (size 1.524 1.524) (drill 1.2) (layers *.Cu *.Mask)
+      (net 6 +3V3))
+    (pad 1 thru_hole circle (at 0 0) (size 1.524 1.524) (drill 1.2) (layers *.Cu *.Mask)
+      (net 6 +3V3))
+    (pad 2 thru_hole circle (at 2.54 2.54) (size 1.524 1.524) (drill 1.2) (layers *.Cu *.Mask)
+      (net 4 /PWM))
+    (pad 2 thru_hole circle (at 2.54 0) (size 1.524 1.524) (drill 1.2) (layers *.Cu *.Mask)
+      (net 4 /PWM))
+    (pad 3 thru_hole circle (at 5.08 2.54) (size 1.524 1.524) (drill 1.2) (layers *.Cu *.Mask)
+      (net 2 GND))
     (pad 3 thru_hole circle (at 5.08 0) (size 1.524 1.524) (drill 1.2) (layers *.Cu *.Mask)
       (net 2 GND))
-    (pad 2 thru_hole circle (at 2.54 0) (size 1.524 1.524) (drill 1.2) (layers *.Cu *.Mask)
-      (net 4 /PWM))
-    (pad 1 thru_hole circle (at 0 0) (size 1.524 1.524) (drill 1.2) (layers *.Cu *.Mask)
-      (net 6 +3V3))
-    (pad 3 thru_hole circle (at 5.08 2.54) (size 1.524 1.524) (drill 1.2) (layers *.Cu *.Mask)
-      (net 2 GND))
-    (pad 2 thru_hole circle (at 2.54 2.54) (size 1.524 1.524) (drill 1.2) (layers *.Cu *.Mask)
-      (net 4 /PWM))
-    (pad 1 thru_hole circle (at 0 2.54) (size 1.524 1.524) (drill 1.2) (layers *.Cu *.Mask)
-      (net 6 +3V3))
   )
   (module Lulu_footprints:LED_Lulu_side (layer F.Cu)
@@
   )
   (module Package_TO_SOT_SMD:SOT-23 (layer F.Cu)
-    (at 124.46 102.87 180)
+    (at 124.206 102.87 180)
     (descr "SOT-23, Standard")
     (tags SOT-23)
@@
   )
   (module Package_TO_SOT_SMD:SOT-23 (layer F.Cu)
-    (at 128.27 102.87)
+    (at 128.016 102.87)
     (descr "SOT-23, Standard")
     (tags SOT-23)
@@
   )
   (module Resistor_SMD:R_0603_1608Metric_Pad1.05x0.95mm_HandSolder (layer F.Cu)
-    (at 125.73 100.33)
+    (at 125.476 100.33)
     (descr "Resistor SMD 0603 (1608 Metric), square (rectangular) end terminal, IPC_7351 nominal with elongated pad for handsoldering. (Body size source: http://www.tortai-tech.com/upload/download/2011102023233369053.pdf), generated with kicad-footprint-generator")
     (tags "resistor handsolder")
