File: Hardware/kicad_Lulu_star/Lulu_star_410/Lulu_star_410.kicad_pcb (KiCad board)
At the start: 2 copper layers, 16.7 x 14.9 mm, 8 parts, among them J1 Conn_01x03_Female, P1 Soldering_pad, Q1 Q_NMOS_GSD, T1 Q_NPN_BEC

Commit message: Start
Parts:
- added U1: ATtiny85-20MU, Package_DFN_QFN:QFN-20-1EP_4x4mm_P0.5mm_EP2.25x2.25mm, F.Cu at (80.8, 34.1)
Connections:
- LED1 pad : GND -> (no net)
