File: Hardware/kicad_Lulu_star/Lulu_star_410/Lulu_star_410.sch (KiCad schematic (older format))
At the start: 6 parts, among them J1 Conn_01x03_Female, Q1 Q_NMOS_GSD, T1 Q_NPN_BEC

Commit message: Start
Parts:
- added R3: 10 K, Resistor_SMD:R_0603_1608Metric_Pad1.05x0.95mm_HandSolder, symbol Device:R
- added U1: ATtiny85-20MU, Package_DFN_QFN:QFN-20-1EP_4x4mm_P0.5mm_EP2.25x2.25mm, symbol MCU_Microchip_ATtiny:ATtiny85-20MU
Connections:
- wire segments 20 -> 23
Changed lines of the file:
@@
 EESchema Schematic File Version 4
-LIBS:Lulu_star_212-cache
+LIBS:Lulu_star_410-cache
 EELAYER 26 0
 EELAYER END
@@
 	-1   0    0    -1
 $EndComp
+Wire Wire Line
+	4850 4050 5150 4050
+Wire Wire Line
+	5800 3700 5800 3850
+Wire Wire Line
+	5800 3250 5800 3400
+Wire Wire Line
+	5800 4250 5800 4400
+Wire Wire Line
+	5450 4400 5800 4400
+Connection ~ 5800 4400
+Wire Wire Line
+	5800 4400 5800 4500
+Wire Wire Line
+	5150 4600 5150 4900
+Wire Wire Line
+	5150 4200 5150 4050
+Connection ~ 5150 4050
+Wire Wire Line
+	5150 4050 5500 4050
+Wire Wire Line
+	5800 4800 5800 4900
+Wire Wire Line
+	5800 4900 5150 4900
+Connection ~ 5150 4900
+Wire Wire Line
+	5150 4900 5150 5000
+Wire Wire Line
+	4550 4050 4350 4050
+Text Label 4100 4050 0    50   ~ 0
+PWM
+Wire Wire Line
+	6000 3550 6700 3550
+Text Label 6350 3550 0    50   ~ 0
+thermal
+Entry Wire Line
+	5800 3550 5900 3650
+$Comp
+L power:GND #PWR0103
+U 1 1 5B7C9260
+P 7050 5000
+F 0 "#PWR0103" H 7050 4750 50  0001 C CNN
+F 1 "GND" H 7055 4827 50  0000 C CNN
+F 2 "" H 7050 5000 50  0001 C CNN
+F 3 "" H 7050 5000 50  0001 C CNN
+	1    7050 5000
+	1    0    0    -1
+$EndComp
+Wire Wire Line
+	7050 5000 7050 4750
+Text Label 7050 4800 0    50   ~ 0
+thermal
+$Comp
+L Connector:Conn_01x03_Female J1
+U 1 1 5B7D3F18
+P 7250 4200
+F 0 "J1" H 7277 4226 50  0000 L CNN
+F 1 "Conn_01x03_Female" H 7277 4135 50  0000 L CNN
+F 2 "Lulu_footprints:Lulu_plug_3" H 7250 4200 50  0001 C CNN
+F 3 "~" H 7250 4200 50  0001 C CNN
+	1    7250 4200
+	1    0    0    -1
+$EndComp
+Wire Wire Line
+	7050 4100 6750 4100
+Wire Wire Line
+	7050 4200 6750 4200
+Wire Wire Line
+	7050 4300 6750 4300
+Text Label 6800 4200 0    50   ~ 0
+PWM
+$Comp
+L power:GND #PWR0104
+U 1 1 5B7D4527
+P 6750 5000
+F 0 "#PWR0104" H 6750 4750 50  0001 C CNN
+F 1 "GND" H 6755 4827 50  0000 C CNN
+F 2 "" H 6750 5000 50  0001 C CNN
+F 3 "" H 6750 5000 50  0001 C CNN
+	1    6750 5000
+	1    0    0    -1
+$EndComp
+Wire Wire Line
+	6750 4300 6750 5000
+$Comp
+L power:+3.3V #PWR0105
+U 1 1 5B7D46B5
+P 6750 3900
+F 0 "#PWR0105" H 6750 3750 50  0001 C CNN
+F 1 "+3.3V" H 6765 4073 50  0000 C CNN
+F 2 "" H 6750 3900 50  0001 C CNN
+F 3 "" H 6750 3900 50  0001 C CNN
+	1    6750 3900
+	1    0    0    -1
+$EndComp
+Wire Wire Line
+	6750 3900 6750 4100
 $Comp
 L Device:R R1
@@
 	0    1    1    0
 $EndComp
-Wire Wire Line
-	4850 4050 5150 4050
-Wire Wire Line
-	5800 3700 5800 3850
-Wire Wire Line
-	5800 3250 5800 3400
-Wire Wire Line
-	5800 4250 5800 4400
-Wire Wire Line
-	5450 4400 5800 4400
-Connection ~ 5800 4400
-Wire Wire Line
-	5800 4400 5800 4500
-Wire Wire Line
-	5150 4600 5150 4900
-Wire Wire Line
-	5150 4200 5150 4050
-Connection ~ 5150 4050
-Wire Wire Line
-	5150 4050 5500 4050
-Wire Wire Line
-	5800 4800 5800 4900
-Wire Wire Line
-	5800 4900 5150 4900
-Connection ~ 5150 4900
-Wire Wire Line
-	5150 4900 5150 5000
-Wire Wire Line
-	4550 4050 4050 4050
-Text Label 4100 4050 0    50   ~ 0
-PWM
-Wire Wire Line
-	6000 3550 6700 3550
-Text Label 6350 3550 0    50   ~ 0
-thermal
-Entry Wire Line
-	5800 3550 5900 3650
-$Comp
-L power:GND #PWR0103
-U 1 1 5B7C9260
-P 7050 5000
-F 0 "#PWR0103" H 7050 4750 50  0001 C CNN
-F 1 "GND" H 7055 4827 50  0000 C CNN
-F 2 "" H 7050 5000 50  0001 C CNN
-F 3 "" H 7050 5000 50  0001 C CNN
-	1    7050 5000
-	1    0    0    -1
-$EndComp
-Wire Wire Line
-	7050 5000 7050 4750
-Text Label 7050 4800 0    50   ~ 0
-thermal
-$Comp
-L Connector:Conn_01x03_Female J1
-U 1 1 5B7D3F18
-P 7250 4200
-F 0 "J1" H 7277 4226 50  0000 L CNN
-F 1 "Conn_01x03_Female" H 7277 4135 50  0000 L CNN
-F 2 "Lulu_footprints:Lulu_plug_3" H 7250 4200 50  0001 C CNN
-F 3 "~" H 7250 4200 50  0001 C CNN
-	1    7250 4200
-	1    0    0    -1
-$EndComp
-Wire Wire Line
-	7050 4100 6750 4100
-Wire Wire Line
-	7050 4200 6750 4200
-Wire Wire Line
-	7050 4300 6750 4300
-Text Label 6800 4200 0    50   ~ 0
-PWM
-$Comp
-L power:GND #PWR0104
-U 1 1 5B7D4527
-P 6750 5000
-F 0 "#PWR0104" H 6750 4750 50  0001 C CNN
-F 1 "GND" H 6755 4827 50  0000 C CNN
-F 2 "" H 6750 5000 50  0001 C CNN
-F 3 "" H 6750 5000 50  0001 C CNN
-	1    6750 5000
-	1    0    0    -1
-$EndComp
-Wire Wire Line
-	6750 4300 6750 5000
-$Comp
-L power:+3.3V #PWR0105
-U 1 1 5B7D46B5
-P 6750 3900
-F 0 "#PWR0105" H 6750 3750 50  0001 C CNN
-F 1 "+3.3V" H 6765 4073 50  0000 C CNN
-F 2 "" H 6750 3900 50  0001 C CNN
-F 3 "" H 6750 3900 50  0001 C CNN
-	1    6750 3900
-	1    0    0    -1
-$EndComp
-Wire Wire Line
-	6750 3900 6750 4100
+$Comp
+L Device:R R3
+U 1 1 5B90D0C4
+P 4350 4400
+F 0 "R3" V 4143 4400 50  0000 C CNN
+F 1 "10 K" V 4234 4400 50  0000 C CNN
+F 2 "Resistor_SMD:R_0603_1608Metric_Pad1.05x0.95mm_HandSolder" V 4280 4400 50  0001 C CNN
+F 3 "~" H 4350 4400 50  0001 C CNN
+	1    4350 4400
+	1    0    0    -1
+$EndComp
+Wire Wire Line
+	4350 4250 4350 4050
+Connection ~ 4350 4050
+Wire Wire Line
+	4350 4050 4050 4050
+$Comp
+L power:GND #PWR0106
+U 1 1 5B90D60D
+P 4350 5000
+F 0 "#PWR0106" H 4350 4750 50  0001 C CNN
+F 1 "GND" H 4355 4827 50  0000 C CNN
+F 2 "" H 4350 5000 50  0001 C CNN
+F 3 "" H 4350 5000 50  0001 C CNN
+	1    4350 5000
+	1    0    0    -1
+$EndComp
+Wire Wire Line
+	4350 4550 4350 5000
+$Comp
+L MCU_Microchip_ATtiny:ATtiny85-20MU U1
+U 1 1 5BA516BD
+P 2650 4150
+F 0 "U1" H 2110 4196 50  0000 R CNN
+F 1 "ATtiny85-20MU" H 2110 4105 50  0000 R CNN
+F 2 "Package_DFN_QFN:QFN-20-1EP_4x4mm_P0.5mm_EP2.25x2.25mm" H 2650 4150 50  0001 C CIN
+F 3 "http://ww1.microchip.com/downloads/en/DeviceDoc/atmel-2586-avr-8-bit-microcontroller-attiny25-attiny45-attiny85_datasheet.pdf" H 2650 4150 50  0001 C CNN
+	1    2650 4150
+	1    0    0    -1
+$EndComp
 $EndSCHEMATC
