File: Hardware/kicad_Lulu_star/Lulu_star_213.kicad_pcb (KiCad board)
At the start: 2 copper layers, 18.6 x 16.3 mm, 8 parts, among them J1 Conn_01x03_Female, P1 Soldering_pad, Q1 Q_NMOS_GSD, T1 Q_NPN_BEC

Commit message: Minor changes
Parts:
- added P1: Soldering_pad, Lulu_footprints:Lulu_brass_tube_pad, F.Cu at (75.3, 39.2)
- moved P1 0.61 mm to (75.3, 39.2)
Changed lines of the file:
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@@
     (tracks 71)
     (zones 0)
-    (modules 8)
+    (modules 9)
     (nets 7)
   )
@@
     (mod_text_size 1 1)
     (mod_text_width 0.15)
-    (pad_size 2.48 2.48)
+    (pad_size 3.5 3.5)
     (pad_drill 0)
     (pad_to_mask_clearance 0)
@@
       (drillshape 0)
       (scaleselection 1)
-      (outputdirectory "Lulu_star_212_GERBER/"))
+      (outputdirectory "Lulu_star_213_GERBER/"))
   )
   (net 0 "")
@@
     (add_net "Net-(Q1-Pad1)")
   )
+  (module Lulu_footprints:Lulu_brass_tube_pad (layer F.Cu)
+    (at 75.33894 39.19982 90)
+    (descr www.etextile.org)
+    (tags eTextile)
+    (zone_connect 1)
+    (attr smd)
+    (fp_text reference P1 (at 0.254 1.143 90) (layer F.SilkS) hide
+      (effects (font (size 1 1) (thickness 0.15)))
+    )
+    (fp_text value Soldering_pad (at -1.018116 -4.840572) (layer F.Fab) hide
+      (effects (font (size 1 1) (thickness 0.15)))
+    )
+    (pad "" smd circle (at 0.01304 -0.02662 120) (size 3.5 3.5) (layers B.Cu B.Paste B.Mask)
+      (net 2 GND) (zone_connect 1) (thermal_gap 0.3))
+  )
   (module Resistor_SMD:R_1206_3216Metric_Pad1.42x1.75mm_HandSolder (layer B.Cu)
     (at 67.11696 37.63772 240)
@@
   )
   (module Lulu_footprints:Lulu_plug_3_spaced (layer F.Cu)
-    (at 69.9135 44.196)
+    (at 69.87286 44.1833)
     (descr www.etextile.org)
     (tags eTextile)
@@
   )
   (module Lulu_footprints:Lulu_brass_tube_pad (layer F.Cu)
-    (at 75.8 39.55 90)
+    (at 75.31232 39.18678 90)
     (descr www.etextile.org)
     (tags eTextile)
@@
       (effects (font (size 1 1) (thickness 0.15)))
     )
-    (pad "" smd circle (at 0 0 90) (size 3.5 3.5) (layers *.Paste *.Mask F.Cu)
-      (net 2 GND) (zone_connect 2))
-  )
-  (gr_text PWM (at 73.40602 43.87728 90) (layer F.SilkS)
-    (effects (font (size 0.7 0.7) (thickness 0.16)))
-  )
-  (gr_text VCC (at 63.21602 44.03728 90) (layer F.SilkS)
-    (effects (font (size 0.7 0.7) (thickness 0.16)))
-  )
-  (gr_text GND (at 68.32102 43.970614 90) (layer F.SilkS)
-    (effects (font (size 0.7 0.7) (thickness 0.16)))
+    (pad "" smd circle (at 0 0 120) (size 3.5 3.5) (layers F.Cu F.Paste F.Mask)
+      (net 2 GND) (zone_connect 1) (thermal_gap 0.3))
   )
   (dimension 16.34998 (width 0.3) (layer F.SilkS)
@@
   )
   (dimension 18.600003 (width 0.3) (layer F.SilkS)
-    (gr_text "18.600 mm" (at 69.837173 50.754031 359.9691958) (layer F.SilkS)
+    (gr_text "18.600 mm" (at 69.796533 50.741331 359.9691958) (layer F.SilkS)
       (effects (font (size 1.5 1.5) (thickness 0.3)))
     )
-    (feature1 (pts (xy 79.14 45.5) (xy 79.137986 49.245451)))
-    (feature2 (pts (xy 60.54 45.49) (xy 60.537986 49.235451)))
-    (crossbar (pts (xy 60.538302 48.649031) (xy 79.138302 48.659031)))
-    (arrow1a (pts (xy 79.138302 48.659031) (xy 78.011483 49.244846)))
-    (arrow1b (pts (xy 79.138302 48.659031) (xy 78.012114 48.072005)))
-    (arrow2a (pts (xy 60.538302 48.649031) (xy 61.66449 49.236057)))
-    (arrow2b (pts (xy 60.538302 48.649031) (xy 61.665121 48.063216)))
+    (feature1 (pts (xy 79.09936 45.4873) (xy 79.097346 49.232751)))
+    (feature2 (pts (xy 60.49936 45.4773) (xy 60.497346 49.222751)))
+    (crossbar (pts (xy 60.497662 48.636331) (xy 79.097662 48.646331)))
+    (arrow1a (pts (xy 79.097662 48.646331) (xy 77.970843 49.232146)))
+    (arrow1b (pts (xy 79.097662 48.646331) (xy 77.971474 48.059305)))
+    (arrow2a (pts (xy 60.497662 48.636331) (xy 61.62385 49.223357)))
+    (arrow2b (pts (xy 60.497662 48.636331) (xy 61.624481 48.050516)))
+  )
+  (gr_text PWM (at 73.36538 43.86458 90) (layer F.SilkS)
+    (effects (font (size 0.7 0.7) (thickness 0.16)))
+  )
+  (gr_text VCC (at 63.17538 44.02458 90) (layer F.SilkS)
+    (effects (font (size 0.7 0.7) (thickness 0.16)))
+  )
+  (gr_text GND (at 68.28038 43.957914 90) (layer F.SilkS)
+    (effects (font (size 0.7 0.7) (thickness 0.16)))
   )
   (gr_line (start 69.8612 29.76223) (end 70.0072 29.64479) (layer Edge.Cuts) (width 0.01))
@@
   (gr_line (start 71.88352 29.18212) (end 72.07855 29.22482) (layer Edge.Cuts) (width 0.01))
   (gr_line (start 69.469 30.1625) (end 69.59204 30.02214) (layer Edge.Cuts) (width 0.01))
-  (gr_text VCC (at 63.22872 44.04744 90) (layer B.SilkS)
+  (gr_text VCC (at 63.18808 44.03474 90) (layer B.SilkS)
     (effects (font (size 0.7 0.7) (thickness 0.16)) (justify mirror))
   )
-  (gr_text PWM (at 73.41872 43.88744 90) (layer B.SilkS)
+  (gr_text PWM (at 73.37808 43.87474 90) (layer B.SilkS)
     (effects (font (size 0.7 0.7) (thickness 0.16)) (justify mirror))
   )
-  (gr_text GND (at 68.33372 43.980774 90) (layer B.SilkS)
+  (gr_text GND (at 68.29308 43.968074 90) (layer B.SilkS)
     (effects (font (size 0.7 0.7) (thickness 0.16)) (justify mirror))
   )
-  (gr_text V.213 (at 72.40016 37.91712 120) (layer B.Mask)
+  (gr_text V.213 (at 71.7042 36.6141 120) (layer B.Mask)
     (effects (font (size 0.9 0.9) (thickness 0.225)) (justify mirror))
   )
-  (gr_text Lulu (at 71.07428 39.72306 120) (layer B.Mask)
+  (gr_text Lulu (at 70.90664 39.80688 120) (layer B.Mask)
     (effects (font (size 2 2) (thickness 0.4)) (justify mirror))
   )
@@
   (segment (start 70.293263 35.36442) (end 68.45046 35.36442) (width 0.25) (layer F.Cu) (net 1))
   (segment (start 71.437362 36.508519) (end 70.293263 35.36442) (width 0.25) (layer F.Cu) (net 1))
-  (via (at 67.3735 44.18) (size 1) (drill 0.8) (layers F.Cu B.Cu) (net 2))
-  (via (at 77.5335 44.18) (size 1) (drill 0.8) (layers F.Cu B.Cu) (net 2))
-  (via (at 62.2935 44.18) (size 1) (drill 0.8) (layers F.Cu B.Cu) (net 2))
-  (via (at 72.4535 44.18) (size 1) (drill 0.8) (layers F.Cu B.Cu) (net 2))
-  (via (at 73.80478 40.77208) (size 0.8) (drill 0.4) (layers F.Cu B.Cu) (net 2))
+  (via (at 67.33286 44.1673) (size 1) (drill 0.8) (layers F.Cu B.Cu) (net 2))
+  (via (at 77.49286 44.1673) (size 1) (drill 0.8) (layers F.Cu B.Cu) (net 2))
+  (via (at 62.25286 44.1673) (size 1) (drill 0.8) (layers F.Cu B.Cu) (net 2))
+  (via (at 72.41286 44.1673) (size 1) (drill 0.8) (layers F.Cu B.Cu) (net 2))
+  (via (at 73.04024 40.26408) (size 0.8) (drill 0.4) (layers F.Cu B.Cu) (net 2))
   (segment (start 69.886706 36.508519) (end 70.00236 36.508519) (width 0.15) (layer F.Cu) (net 3))
   (segment (start 70.00236 36.508519) (end 70.00236 36.558519) (width 0.15) (layer F.Cu) (net 3))
