File: Hardware/kicad_Lulu_MCU/Lulu_MCU_4.0.0.kicad_pcb (KiCad board)
At the start: 2 copper layers, 18.6 x 16.3 mm, 9 parts, among them J1 Conn_01x03_Female, P1 Soldering_pad, Q1 Q_NMOS_GSD, T1 Q_NPN_BEC

Commit message: Routing in process
Parts:
- removed P1 (x2): Soldering_pad, Lulu_footprints:Lulu_brass_tube_pad
- added U1: ATtiny10-TS, Package_TO_SOT_SMD:SOT-23-6, F.Cu at (68.2, 41.8)
- J1: footprint Lulu_footprints:Lulu_plug_3_spaced -> Lulu_footprints:Lulu_brass_tube_pad
- R1: value 47K -> 47 K
- R3: value 10K -> 10 K
- moved J1 7.53 mm to (75.4, 39.1)
Connections:
- LED1 pad : GND -> (no net)
Routing:
- net /PWM: track 11.6 -> 2.36 mm
Changed lines of the file:
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@@
     (thickness 1)
     (drawings 49)
-    (tracks 71)
+    (tracks 65)
     (zones 0)
-    (modules 9)
-    (nets 7)
+    (modules 8)
+    (nets 10)
   )
   (page User 148.488 105.004)
@@
     (32 B.Adhes user)
     (33 F.Adhes user)
-    (34 B.Paste user hide)
+    (34 B.Paste user)
     (35 F.Paste user)
     (36 B.SilkS user)
-    (37 F.SilkS user hide)
+    (37 F.SilkS user)
     (38 B.Mask user)
     (39 F.Mask user)
@@
     (45 Margin user)
     (46 B.CrtYd user)
-    (47 F.CrtYd user hide)
-    (48 B.Fab user hide)
+    (47 F.CrtYd user)
+    (48 B.Fab user)
     (49 F.Fab user)
   )
@@
   (net 5 "Net-(LED1-Pad1)")
   (net 6 +3V3)
+  (net 7 /DATA)
+  (net 8 "Net-(U1-Pad6)")
+  (net 9 /SENSOR)
   (net_class Default "This is the default net class."
     (clearance 0.2)
@@
     (uvia_dia 0.3)
     (uvia_drill 0.1)
+    (add_net /DATA)
+    (add_net /SENSOR)
     (add_net GND)
     (add_net "Net-(Q1-Pad2)")
+    (add_net "Net-(U1-Pad6)")
   )
   (net_class POWER ""
@@
   )
   (module Lulu_footprints:Lulu_brass_tube_pad (layer F.Cu)
-    (at 75.33894 39.19982 90)
+    (at 75.40244 39.0779)
     (descr www.etextile.org)
     (tags eTextile)
     (zone_connect 1)
     (attr smd)
-    (fp_text reference P1 (at 0.254 1.143 90) (layer F.SilkS) hide
-      (effects (font (size 1 1) (thickness 0.15)))
-    )
-    (fp_text value Soldering_pad (at -1.018116 -4.840572) (layer F.Fab) hide
-      (effects (font (size 1 1) (thickness 0.15)))
-    )
-    (pad "" smd circle (at 0.01304 -0.02662 120) (size 3.5 3.5) (layers B.Cu B.Paste B.Mask)
-      (net 2 GND) (zone_connect 1) (thermal_gap 0.3))
+    (fp_text reference J1 (at 0.254 1.143) (layer F.SilkS) hide
+      (effects (font (size 1 1) (thickness 0.15)))
+    )
+    (fp_text value Conn_01x03_Female (at -1.018116 -4.840572 -90) (layer F.Fab) hide
+      (effects (font (size 1 1) (thickness 0.15)))
+    )
+    (pad 1 smd circle (at 0 0) (size 3.5 3.5) (layers *.Paste *.Mask F.Cu)
+      (net 6 +3V3) (zone_connect 1))
+  )
+  (module Package_TO_SOT_SMD:SOT-23-6 (layer F.Cu)
+    (at 68.23456 41.84904)
+    (descr "6-pin SOT-23 package")
+    (tags SOT-23-6)
+    (attr smd)
+    (fp_text reference U1 (at 0 -2.9) (layer F.SilkS)
+      (effects (font (size 1 1) (thickness 0.15)))
+    )
+    (fp_text value ATtiny10-TS (at 0 2.9) (layer F.Fab)
+      (effects (font (size 1 1) (thickness 0.15)))
+    )
+    (fp_text user %R (at 0 0 90) (layer F.Fab)
+      (effects (font (size 0.5 0.5) (thickness 0.075)))
+    )
+    (fp_line (start -0.9 1.61) (end 0.9 1.61) (layer F.SilkS) (width 0.12))
+    (fp_line (start 0.9 -1.61) (end -1.55 -1.61) (layer F.SilkS) (width 0.12))
+    (fp_line (start 1.9 -1.8) (end -1.9 -1.8) (layer F.CrtYd) (width 0.05))
+    (fp_line (start 1.9 1.8) (end 1.9 -1.8) (layer F.CrtYd) (width 0.05))
+    (fp_line (start -1.9 1.8) (end 1.9 1.8) (layer F.CrtYd) (width 0.05))
+    (fp_line (start -1.9 -1.8) (end -1.9 1.8) (layer F.CrtYd) (width 0.05))
+    (fp_line (start -0.9 -0.9) (end -0.25 -1.55) (layer F.Fab) (width 0.1))
+    (fp_line (start 0.9 -1.55) (end -0.25 -1.55) (layer F.Fab) (width 0.1))
+    (fp_line (start -0.9 -0.9) (end -0.9 1.55) (layer F.Fab) (width 0.1))
+    (fp_line (start 0.9 1.55) (end -0.9 1.55) (layer F.Fab) (width 0.1))
+    (fp_line (start 0.9 -1.55) (end 0.9 1.55) (layer F.Fab) (width 0.1))
+    (pad 1 smd rect (at -1.1 -0.95) (size 1.06 0.65) (layers F.Cu F.Paste F.Mask)
+      (net 9 /SENSOR))
+    (pad 2 smd rect (at -1.1 0) (size 1.06 0.65) (layers F.Cu F.Paste F.Mask)
+      (net 2 GND))
+    (pad 3 smd rect (at -1.1 0.95) (size 1.06 0.65) (layers F.Cu F.Paste F.Mask)
+      (net 4 /PWM))
+    (pad 4 smd rect (at 1.1 0.95) (size 1.06 0.65) (layers F.Cu F.Paste F.Mask)
+      (net 7 /DATA))
+    (pad 6 smd rect (at 1.1 -0.95) (size 1.06 0.65) (layers F.Cu F.Paste F.Mask)
+      (net 8 "Net-(U1-Pad6)"))
+    (pad 5 smd rect (at 1.1 0) (size 1.06 0.65) (layers F.Cu F.Paste F.Mask)
+      (net 6 +3V3))
+    (model ${KISYS3DMOD}/Package_TO_SOT_SMD.3dshapes/SOT-23-6.wrl
+      (at (xyz 0 0 0))
+      (scale (xyz 1 1 1))
+      (rotate (xyz 0 0 0))
+    )
   )
   (module Resistor_SMD:R_1206_3216Metric_Pad1.42x1.75mm_HandSolder (layer B.Cu)
@@
     )
   )
-  (module Lulu_footprints:Lulu_plug_3_spaced (layer F.Cu)
-    (at 69.87286 44.1833)
-    (descr www.etextile.org)
-    (tags eTextile)
-    (zone_connect 0)
-    (fp_text reference J1 (at 0 -2.921) (layer F.SilkS) hide
-      (effects (font (size 1 1) (thickness 0.15)))
-    )
-    (fp_text value Conn_01x03_Female (at 0 3.175) (layer F.Fab) hide
-      (effects (font (size 1 1) (thickness 0.15)))
-    )
-    (pad 3 smd roundrect (at 5.08 0) (size 2 4.6) (layers F.Cu F.Mask) (roundrect_rratio 0.5)
-      (net 4 /PWM) (zone_connect 2))
-    (pad 3 thru_hole circle (at 5.08 -1.3) (size 2 2) (drill 1.4) (layers *.Cu *.Mask)
-      (net 4 /PWM) (zone_connect 2))
-    (pad 3 thru_hole circle (at 5.08 1.3) (size 2 2) (drill 1.4) (layers *.Cu *.Mask)
-      (net 4 /PWM) (zone_connect 2))
-    (pad 2 thru_hole circle (at 0 -1.3) (size 2 2) (drill 1.4) (layers *.Cu *.Mask)
-      (net 2 GND) (zone_connect 2))
-    (pad 2 smd roundrect (at 0 0) (size 2 4.6) (layers F.Cu F.Mask) (roundrect_rratio 0.5)
-      (net 2 GND) (zone_connect 2))
-    (pad 2 thru_hole circle (at 0 1.3) (size 2 2) (drill 1.4) (layers *.Cu *.Mask)
-      (net 2 GND) (zone_connect 2))
-    (pad 1 smd roundrect (at -5.08 0) (size 2 4.6) (layers F.Cu F.Mask) (roundrect_rratio 0.5)
-      (net 6 +3V3) (zone_connect 2))
-    (pad 1 thru_hole circle (at -5.08 1.3) (size 2 2) (drill 1.4) (layers *.Cu *.Mask)
-      (net 6 +3V3) (zone_connect 2))
-    (pad 1 thru_hole circle (at -5.08 -1.3) (size 2 2) (drill 1.4) (layers *.Cu *.Mask)
-      (net 6 +3V3) (zone_connect 2))
-    (pad 3 smd roundrect (at 5.08 0) (size 2 4.6) (layers B.Cu B.Mask) (roundrect_rratio 0.5)
-      (net 4 /PWM) (zone_connect 2))
-    (pad 1 smd roundrect (at -5.08 0) (size 2 4.6) (layers B.Cu B.Mask) (roundrect_rratio 0.5)
-      (net 6 +3V3) (zone_connect 2))
-    (pad 2 smd roundrect (at 0 0) (size 2 4.6) (layers B.Cu B.Mask) (roundrect_rratio 0.5)
-      (net 2 GND) (zone_connect 2))
-  )
   (module Lulu_footprints:Lulu_side_LED (layer F.Cu)
     (at 74.64 35.4 30)
@@
     (fp_poly (pts (xy -1.1 0.6) (xy 1.1 0.6) (xy 1.1 10.6) (xy -1.1 10.6)) (layer F.Fab) (width 0))
     (pad "" smd custom (at -0.685801 -5.065372 30) (size 2.48 2.48) (layers B.Cu B.Mask)
-      (net 2 GND) (zone_connect 2)
+      (zone_connect 2)
       (options (clearance outline) (anchor circle))
       (primitives
@@
       ))
     (pad "" smd custom (at -0.685801 -5.065372 30) (size 2.48 2.48) (layers F.Cu F.Mask)
-      (net 2 GND) (zone_connect 2)
+      (zone_connect 2)
       (options (clearance outline) (anchor circle))
       (primitives
@@
       (effects (font (size 1 1) (thickness 0.15)))
     )
-    (fp_text value 10K (at 4.83616 0.01524 180) (layer F.Fab)
+    (fp_text value "10 K" (at 4.83616 0.01524 180) (layer F.Fab)
       (effects (font (size 1 1) (thickness 0.15)))
     )
@@
       (effects (font (size 1 1) (thickness 0.15)))
     )
-    (fp_text value 47K (at 3.93192 0.03556 180) (layer F.Fab)
+    (fp_text value "47 K" (at 3.93192 0.03556 180) (layer F.Fab)
       (effects (font (size 1 1) (thickness 0.15)))
     )
@@
       (rotate (xyz 0 0 0))
     )
-  )
-  (module Lulu_footprints:Lulu_brass_tube_pad (layer F.Cu)
-    (at 75.31232 39.18678 90)
-    (descr www.etextile.org)
-    (tags eTextile)
-    (zone_connect 1)
-    (attr smd)
-    (fp_text reference P1 (at 0.254 1.143 90) (layer F.SilkS) hide
-      (effects (font (size 1 1) (thickness 0.15)))
-    )
-    (fp_text value Soldering_pad (at -1.018116 -4.840572) (layer F.Fab) hide
-      (effects (font (size 1 1) (thickness 0.15)))
-    )
-    (pad "" smd circle (at 0 0 120) (size 3.5 3.5) (layers F.Cu F.Paste F.Mask)
-      (net 2 GND) (zone_connect 1) (thermal_gap 0.3))
   )
   (dimension 16.34998 (width 0.3) (layer F.SilkS)
@@
   (segment (start 67.71002 37.89426) (end 68.44408 38.62832) (width 0.15) (layer F.Cu) (net 4))
   (segment (start 67.42306 37.89426) (end 67.71002 37.89426) (width 0.15) (layer F.Cu) (net 4))
-  (segment (start 68.44408 40.26024) (end 68.44408 38.62832) (width 0.15) (layer F.Cu) (net 4))
-  (segment (start 70.57898 41.56964) (end 69.75348 41.56964) (width 0.15) (layer F.Cu) (net 4))
-  (segment (start 71.00062 41.99128) (end 70.57898 41.56964) (width 0.15) (layer F.Cu) (net 4))
-  (segment (start 74.9935 42.896) (end 74.08878 41.99128) (width 0.15) (layer F.Cu) (net 4))
-  (segment (start 69.75348 41.56964) (end 68.44408 40.26024) (width 0.15) (layer F.Cu) (net 4))
-  (segment (start 74.08878 41.99128) (end 71.00062 41.99128) (width 0.15) (layer F.Cu) (net 4))
   (segment (start 71.45258 35.57) (end 73.43 35.57) (width 0.25) (layer F.Cu) (net 5))
   (segment (start 70.95236 34.508519) (end 70.95236 35.06978) (width 0.25) (layer F.Cu) (net 5))
@@
     (connect_pads yes (clearance 0.4))
     (min_thickness 0.254)
-    (fill yes (arc_segments 32) (thermal_gap 0.508) (thermal_bridge_width 0.508) (smoothing fillet))
+    (fill (arc_segments 32) (thermal_gap 0.508) (thermal_bridge_width 0.508) (smoothing fillet))
     (polygon
       (pts
@@
     (connect_pads yes (clearance 0.4))
     (min_thickness 0.254)
-    (fill yes (arc_segments 32) (thermal_gap 0.508) (thermal_bridge_width 0.508))
+    (fill (arc_segments 32) (thermal_gap 0.508) (thermal_bridge_width 0.508))
     (polygon
       (pts

Commit message: Routing, work in progress
Parts:
- added TP1: TPI_DATA, TestPoint:TestPoint_Pad_D1.0mm, B.Cu at (55.6, 48.0)
- added TP2: TPI_CLOCK, TestPoint:TestPoint_Pad_D1.0mm, B.Cu at (53.4, 48.0)
- added TP3: TPI_RESET, TestPoint:TestPoint_Pad_D1.0mm, B.Cu at (47.0, 48.1)
- added TP4: TPI_VTARGET, TestPoint:TestPoint_Pad_D1.0mm, B.Cu at (49.1, 48.1)
- added TP5: TPI_GND, TestPoint:TestPoint_Pad_D1.0mm, B.Cu at (51.1, 48.1)
- J1: footprint Lulu_footprints:Lulu_brass_tube_pad -> Lulu_footprints:Lulu_plug_3_spaced
- R2: moved to F.Cu
- moved J1 7.68 mm to (69.8, 44.4)
- moved R2 6.22 mm to (62.7, 33.2), turned to 120 degrees
- turned LED1 to 90 degrees
- turned U1 to 90 degrees
Connections:
- R1 pad 2: /PWM -> Net-(R1-Pad2)
- R3 pad 1: /PWM -> Net-(R1-Pad2)
- U1 pad 4: /DATA -> /1-WIRE
- U1 pad 6: Net-(U1-Pad6) -> /RESET
Routing:
- net Net-(R1-Pad2): track 0.00 -> 2.36 mm
- net /PWM: track 2.36 -> 0.00 mm

Commit message: Under routing
Parts:
- moved R1 19.7 mm to (48.5, 32.1)
- moved R3 19.7 mm to (48.5, 33.5)
- moved T1 19.7 mm to (51.9, 33.8)
- moved Q1 19.7 mm to (51.9, 30.4)
- moved U1 12.4 mm to (55.9, 40.6)
- moved R2 5.32 mm to (62.2, 27.9), turned to 0 degrees
- moved LED1 0.33 mm to (74.9, 35.6)
Routing:
- net Net-(Q1-Pad2): track 6.73 -> 0.00 mm, vias 1 -> 0
- net Net-(LED1-Pad1): track 3.25 -> 9.98 mm, vias 0 -> 1
- net GND: vias 5 -> 4
- net /PWM: vias 0 -> 1
Other:
- board size 18.6 x 16.3 mm -> 30.9 x 16.6 mm
Changed lines of the file:
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@@
-(kicad_pcb (version 20171130) (host pcbnew 5.0.2-bee76a0~70~ubuntu18.04.1)
+(kicad_pcb (version 20171130) (host pcbnew 5.0.2+dfsg1-1~bpo9+1)
   (general
     (thickness 1)
-    (drawings 49)
+    (drawings 53)
     (tracks 65)
     (zones 0)
@@
   )
   (layers
-    (0 F.Cu jumper)
-    (31 B.Cu signal)
+    (0 F.Cu jumper hide)
+    (31 B.Cu signal hide)
     (32 B.Adhes user)
     (33 F.Adhes user)
@@
     (36 B.SilkS user)
     (37 F.SilkS user)
-    (38 B.Mask user)
+    (38 B.Mask user hide)
     (39 F.Mask user)
     (40 Dwgs.User user)
     (41 Cmts.User user)
-    (42 Eco1.User user)
+    (42 Eco1.User user hide)
     (43 Eco2.User user)
     (44 Edge.Cuts user)
@@
   )
   (module Package_TO_SOT_SMD:SOT-23-6 (layer F.Cu)
-    (at 68.23456 41.84904 90)
+    (at 55.88 40.64 90)
     (descr "6-pin SOT-23 package")
     (tags SOT-23-6)
@@
   )
   (module Resistor_SMD:R_1206_3216Metric_Pad1.42x1.75mm_HandSolder (layer F.Cu)
-    (at 62.71514 33.24098 120)
+    (at 62.23 27.94)
     (descr "Resistor SMD 1206 (3216 Metric), square (rectangular) end terminal, IPC_7351 nominal with elongated pad for handsoldering. (Body size source: http://www.tortai-tech.com/upload/download/2011102023233369053.pdf), generated with kicad-footprint-generator")
     (tags "resistor handsolder")
     (attr smd)
-    (fp_text reference R2 (at 1.516269 2.209906 30) (layer F.SilkS)
+    (fp_text reference R2 (at 1.516269 2.209906 -90) (layer F.SilkS)
       (effects (font (size 0.7 0.7) (thickness 0.12)))
     )
-    (fp_text value "2.7 Ohm" (at -0.68 -2.52 120) (layer F.Fab)
-      (effects (font (size 1 1) (thickness 0.15)))
-    )
-    (fp_text user %R (at 0 0 120) (layer F.Fab)
+    (fp_text value "2.7 Ohm" (at -0.68 -2.52) (layer F.Fab)
+      (effects (font (size 1 1) (thickness 0.15)))
+    )
+    (fp_text user %R (at 0 0) (layer F.Fab)
       (effects (font (size 0.8 0.8) (thickness 0.12)))
     )
@@
     (fp_line (start -1.6 -0.8) (end 1.6 -0.8) (layer F.Fab) (width 0.1))
     (fp_line (start -1.6 0.8) (end -1.6 -0.8) (layer F.Fab) (width 0.1))
-    (pad 2 smd roundrect (at 1.4875 0 120) (size 1.425 1.75) (layers F.Cu F.Paste F.Mask) (roundrect_rratio 0.175)
+    (pad 2 smd roundrect (at 1.4875 0) (size 1.425 1.75) (layers F.Cu F.Paste F.Mask) (roundrect_rratio 0.175)
       (net 2 GND) (zone_connect 1))
-    (pad 1 smd roundrect (at -1.4875 0 120) (size 1.425 1.75) (layers F.Cu F.Paste F.Mask) (roundrect_rratio 0.175439)
+    (pad 1 smd roundrect (at -1.4875 0) (size 1.425 1.75) (layers F.Cu F.Paste F.Mask) (roundrect_rratio 0.175439)
       (net 1 "Net-(Q1-Pad2)"))
     (model ${KISYS3DMOD}/Resistor_SMD.3dshapes/R_1206_3216Metric.wrl
@@
   )
   (module Lulu_footprints:Lulu_side_LED (layer F.Cu)
-    (at 74.64 35.4 90)
+    (at 74.93 35.56 90)
     (descr "LED Cree-XP http://www.cree.com/~/media/Files/Cree/LED-Components-and-Modules/XLamp/Data-and-Binning/XLampXPE2.pdf")
     (tags "LED Cree XP")
@@
   )
   (module Resistor_SMD:R_0603_1608Metric_Pad1.05x0.95mm_HandSolder (layer F.Cu)
-    (at 67.56908 38.62832 180)
+    (at 48.51908 33.54832 180)
     (descr "Resistor SMD 0603 (1608 Metric), square (rectangular) end terminal, IPC_7351 nominal with elongated pad for handsoldering. (Body size source: http://www.tortai-tech.com/upload/download/2011102023233369053.pdf), generated with kicad-footprint-generator")
     (tags "resistor handsolder")
@@
   )
   (module Package_TO_SOT_SMD:SOT-23 (layer F.Cu)
-    (at 70.95236 38.92804 270)
+    (at 51.90236 33.84804 270)
     (descr "SOT-23, Standard")
     (tags SOT-23)
@@
   )
   (module Package_TO_SOT_SMD:SOT-23 (layer F.Cu)
-    (at 70.95236 35.508519 90)
+    (at 51.90236 30.428519 90)
     (descr "SOT-23, Standard")
     (tags SOT-23)
@@
   )
   (module Resistor_SMD:R_0603_1608Metric_Pad1.05x0.95mm_HandSolder (layer F.Cu)
-    (at 67.56908 37.16528 180)
+    (at 48.51908 32.08528 180)
     (descr "Resistor SMD 0603 (1608 Metric), square (rectangular) end terminal, IPC_7351 nominal with elongated pad for handsoldering. (Body size source: http://www.tortai-tech.com/upload/download/2011102023233369053.pdf), generated with kicad-footprint-generator")
     (tags "resistor handsolder")
@@
     )
   )
-  (dimension 16.34998 (width 0.3) (layer F.SilkS)
-    (gr_text "16.350 mm" (at 54.357736 37.315483 89.99109899) (layer F.SilkS)
+  (gr_line (start 91.44 45.72) (end 85.09 45.72) (layer Edge.Cuts) (width 0.2))
+  (gr_line (start 91.44 38.1) (end 91.44 45.72) (layer Edge.Cuts) (width 0.2))
+  (gr_line (start 85.09 38.1) (end 91.44 38.1) (layer Edge.Cuts) (width 0.2))
+  (gr_line (start 85.09 45.72) (end 85.09 38.1) (layer Edge.Cuts) (width 0.02))
+  (dimension 16.34998 (width 0.3) (layer Eco1.User)
+    (gr_text "16.350 mm" (at 54.357736 37.315483 89.99109899) (layer Eco1.User)
       (effects (font (size 1.5 1.5) (thickness 0.3)))
     )
@@
     (arrow2b (pts (xy 56.459006 29.140819) (xy 57.045252 30.267414)))
   )
-  (dimension 18.600003 (width 0.3) (layer F.SilkS)
-    (gr_text "18.600 mm" (at 69.796533 50.741331 359.9691958) (layer F.SilkS)
+  (dimension 18.600003 (width 0.3) (layer Eco1.User)
+    (gr_text "18.600 mm" (at 69.796533 50.741331 359.9691958) (layer Eco1.User)
       (effects (font (size 1.5 1.5) (thickness 0.3)))
     )
@@
     (effects (font (size 2 2) (thickness 0.4)) (justify mirror))
   )
-  (segment (start 71.90236 36.508519) (end 71.90236 37.92804) (width 0.25) (layer F.Cu) (net 1))
-  (segment (start 71.437362 36.508519) (end 71.90236 36.508519) (width 0.25) (layer F.Cu) (net 1))
-  (via (at 68.45046 35.36442) (size 0.8) (drill 0.4) (layers F.Cu B.Cu) (net 1))
-  (segment (start 68.45046 35.36442) (end 68.62064 35.19424) (width 0.25) (layer F.Cu) (net 1))
-  (segment (start 68.45046 35.36442) (end 67.86071 36.349507) (width 0.25) (layer B.Cu) (net 1))
-  (segment (start 70.293263 35.36442) (end 68.45046 35.36442) (width 0.25) (layer F.Cu) (net 1))
-  (segment (start 71.437362 36.508519) (end 70.293263 35.36442) (width 0.25) (layer F.Cu) (net 1))
+  (segment (start 71.90236 36.508519) (end 71.90236 37.92804) (width 0.25) (layer F.Cu) (net 5))
+  (segment (start 71.437362 36.508519) (end 71.90236 36.508519) (width 0.25) (layer F.Cu) (net 5))
+  (via (at 68.45046 35.36442) (size 0.8) (drill 0.4) (layers F.Cu B.Cu) (net 5))
+  (segment (start 68.45046 35.36442) (end 68.62064 35.19424) (width 0.25) (layer F.Cu) (net 5))
+  (segment (start 68.45046 35.36442) (end 67.86071 36.349507) (width 0.25) (layer B.Cu) (net 5))
+  (segment (start 70.293263 35.36442) (end 68.45046 35.36442) (width 0.25) (layer F.Cu) (net 5))
+  (segment (start 71.437362 36.508519) (end 70.293263 35.36442) (width 0.25) (layer F.Cu) (net 5))
   (via (at 67.33286 44.1673) (size 1.4) (drill 1) (layers F.Cu B.Cu) (net 2))
   (via (at 77.49286 44.1673) (size 1.4) (drill 1) (layers F.Cu B.Cu) (net 2))
   (via (at 62.25286 44.1673) (size 1.4) (drill 1) (layers F.Cu B.Cu) (net 2))
   (via (at 72.41286 44.1673) (size 1.4) (drill 1) (layers F.Cu B.Cu) (net 2))
-  (via (at 73.04024 40.26408) (size 0.8) (drill 0.4) (layers F.Cu B.Cu) (net 2))
+  (via (at 73.04024 40.26408) (size 0.8) (drill 0.4) (layers F.Cu B.Cu) (net 4))
   (segment (start 69.886706 36.508519) (end 70.00236 36.508519) (width 0.15) (layer F.Cu) (net 3))
   (segment (start 70.00236 36.508519) (end 70.00236 36.558519) (width 0.15) (layer F.Cu) (net 3))
@@
   (segment (start 69.345599 37.16528) (end 70.00236 36.508519) (width 0.15) (layer F.Cu) (net 3))
   (segment (start 68.44408 37.16528) (end 69.345599 37.16528) (width 0.15) (layer F.Cu) (net 3))
-  (segment (start 66.69408 37.16528) (end 67.42306 37.89426) (width 0.15) (layer F.Cu) (net 9))
-  (segment (start 67.71002 37.89426) (end 68.44408 38.62832) (width 0.15) (layer F.Cu) (net 9))
-  (segment (start 67.42306 37.89426) (end 67.71002 37.89426) (width 0.15) (layer F.Cu) (net 9))
   (segment (start 71.45258 35.57) (end 73.43 35.57) (width 0.25) (layer F.Cu) (net 5))
   (segment (start 70.95236 34.508519) (end 70.95236 35.06978) (width 0.25) (layer F.Cu) (net 5))
@@
   (segment (start 69.722563 30.373875) (end 69.834202 30.24652) (width 0.25) (layer B.Cu) (net 6))
   (segment (start 69.834202 30.24652) (end 69.952266 30.125949) (width 0.25) (layer B.Cu) (net 6))
+  (segment (start 66.69408 37.16528) (end 67.42306 37.89426) (width 0.15) (layer F.Cu) (net 9))
+  (segment (start 67.71002 37.89426) (end 68.44408 38.62832) (width 0.15) (layer F.Cu) (net 9))
+  (segment (start 67.42306 37.89426) (end 67.71002 37.89426) (width 0.15) (layer F.Cu) (net 9))
   (zone (net 2) (net_name GND) (layer F.Cu) (hatch none 0.508)
     (connect_pads yes (clearance 0.4))
     (min_thickness 0.254)
-    (fill (arc_segments 32) (thermal_gap 0.508) (thermal_bridge_width 0.508) (smoothing fillet))
+    (fill yes (arc_segments 32) (thermal_gap 0.508) (thermal_bridge_width 0.508) (smoothing fillet))
     (polygon
       (pts
@@
     (connect_pads yes (clearance 0.4))
     (min_thickness 0.254)
-    (fill (arc_segments 32) (thermal_gap 0.508) (thermal_bridge_width 0.508))
+    (fill yes (arc_segments 32) (thermal_gap 0.508) (thermal_bridge_width 0.508))
     (polygon
       (pts
