File: Hardware/kicad_Lulu_MCU/Lulu_MCU_4.0.0.sch (KiCad schematic (older format))
At the start: 7 parts, among them J1 Conn_01x03_Female, Q1 Q_NMOS_GSD, T1 Q_NPN_BEC

Commit message: Routing in process
Parts:
- added U1: ATtiny10-TS, Package_TO_SOT_SMD:SOT-23-6, symbol MCU_Microchip_ATtiny:ATtiny10-TS
Connections:
- net labels added: DATA, SENSOR
- wire segments 23 -> 29
Other:
- moved on the sheet: J1, LED1, Q1, R1, R2, R3, T1

Commit message: Routing, work in progress
Parts:
- added TP1: TPI_DATA, TestPoint:TestPoint_Pad_D1.0mm, symbol Connector:TestPoint
- added TP2: TPI_CLOCK, TestPoint:TestPoint_Pad_D1.0mm, symbol Connector:TestPoint
- added TP3: TPI_RESET, TestPoint:TestPoint_Pad_D1.0mm, symbol Connector:TestPoint
- added TP4: TPI_VTARGET, TestPoint:TestPoint_Pad_D1.0mm, symbol Connector:TestPoint
- added TP5: TPI_GND, TestPoint:TestPoint_Pad_D1.0mm, symbol Connector:TestPoint
- J1: footprint Lulu_footprints:Lulu_brass_tube_pad -> Lulu_footprints:Lulu_plug_3_spaced
Connections:
- net labels added: 1-WIRE, RESET
- net labels removed: DATA
- wire segments 29 -> 36
Changed lines of the file:
@@
 Wire Wire Line
 	5650 3700 5450 3700
-Text Label 5200 3700 0    50   ~ 0
+Text Label 4950 3700 0    50   ~ 0
 PWM
 Wire Wire Line
@@
 F 0 "J1" H 8377 3876 50  0000 L CNN
 F 1 "Conn_01x03_Female" H 8377 3785 50  0000 L CNN
-F 2 "Lulu_footprints:Lulu_brass_tube_pad" H 8350 3850 50  0001 C CNN
+F 2 "Lulu_footprints:Lulu_plug_3_spaced" H 8350 3850 50  0001 C CNN
 F 3 "~" H 8350 3850 50  0001 C CNN
 	1    8350 3850
@@
 	8150 3750 7850 3750
 Text Label 7850 3950 0    50   ~ 0
-DATA
+1-WIRE
 $Comp
 L power:GND #PWR0104
@@
 Wire Wire Line
 	5450 3900 5450 3700
-Connection ~ 5450 3700
 Wire Wire Line
 	5450 3700 5150 3700
@@
 SENSOR
 Text Label 4100 3350 0    50   ~ 0
-DATA
+1-WIRE
 Text Label 4100 3250 0    50   ~ 0
 PWM
+$Comp
+L Connector:TestPoint TP1
+U 1 1 5CAD390A
+P 5050 2400
+F 0 "TP1" V 5245 2474 50  0001 C CNN
+F 1 "TPI_DATA" V 5089 2991 50  0000 R BNN
+F 2 "TestPoint:TestPoint_Pad_D1.0mm" H 5250 2400 50  0001 C CNN
+F 3 "~" H 5250 2400 50  0001 C CNN
+	1    5050 2400
+	0    -1   -1   0
+$EndComp
+$Comp
+L Connector:TestPoint TP2
+U 1 1 5CAD39E3
+P 5050 2500
+F 0 "TP2" V 5245 2574 50  0001 C CNN
+F 1 "TPI_CLOCK" V 5089 3091 50  0000 R BNN
+F 2 "TestPoint:TestPoint_Pad_D1.0mm" H 5250 2500 50  0001 C CNN
+F 3 "~" H 5250 2500 50  0001 C CNN
+	1    5050 2500
+	0    -1   -1   0
+$EndComp
+$Comp
+L Connector:TestPoint TP3
+U 1 1 5CADD00C
+P 5050 2600
+F 0 "TP3" V 5245 2674 50  0001 C CNN
+F 1 "TPI_RESET" V 5089 3191 50  0000 R BNN
+F 2 "TestPoint:TestPoint_Pad_D1.0mm" H 5250 2600 50  0001 C CNN
+F 3 "~" H 5250 2600 50  0001 C CNN
+	1    5050 2600
+	0    -1   -1   0
+$EndComp
+$Comp
+L Connector:TestPoint TP4
+U 1 1 5CADD036
+P 5050 2700
+F 0 "TP4" V 5245 2774 50  0001 C CNN
+F 1 "TPI_VTARGET" V 5089 3291 50  0000 R BNN
+F 2 "TestPoint:TestPoint_Pad_D1.0mm" H 5250 2700 50  0001 C CNN
+F 3 "~" H 5250 2700 50  0001 C CNN
+	1    5050 2700
+	0    -1   -1   0
+$EndComp
+$Comp
+L Connector:TestPoint TP5
+U 1 1 5CADD062
+P 5050 2800
+F 0 "TP5" V 5245 2874 50  0001 C CNN
+F 1 "TPI_GND" V 5089 3391 50  0000 R BNN
+F 2 "TestPoint:TestPoint_Pad_D1.0mm" H 5250 2800 50  0001 C CNN
+F 3 "~" H 5250 2800 50  0001 C CNN
+	1    5050 2800
+	0    -1   -1   0
+$EndComp
+Wire Wire Line
+	5050 2500 5300 2500
+Wire Wire Line
+	5050 2600 5300 2600
+$Comp
+L power:+3.3V #PWR?
+U 1 1 5CADF790
+P 5700 2350
+F 0 "#PWR?" H 5700 2200 50  0001 C CNN
+F 1 "+3.3V" H 5715 2523 50  0000 C CNN
+F 2 "" H 5700 2350 50  0001 C CNN
+F 3 "" H 5700 2350 50  0001 C CNN
+	1    5700 2350
+	1    0    0    -1
+$EndComp
+Wire Wire Line
+	5700 2350 5700 2700
+Wire Wire Line
+	5050 2700 5700 2700
+Text Label 4100 3450 0    50   ~ 0
+RESET
+Text Label 5300 2600 0    50   ~ 0
+RESET
+Connection ~ 5450 3700
+Text Label 5300 2500 0    50   ~ 0
+PWM
+Wire Wire Line
+	5700 2950 5700 2800
+Wire Wire Line
+	5700 2800 5050 2800
+$Comp
+L power:GND #PWR?
+U 1 1 5CAE1CC2
+P 5700 2950
+F 0 "#PWR?" H 5700 2700 50  0001 C CNN
+F 1 "GND" H 5705 2777 50  0000 C CNN
+F 2 "" H 5700 2950 50  0001 C CNN
+F 3 "" H 5700 2950 50  0001 C CNN
+	1    5700 2950
+	1    0    0    -1
+$EndComp
+Wire Wire Line
+	5050 2400 5300 2400
+Text Label 5300 2400 0    50   ~ 0
+SENSOR
 $EndSCHEMATC

Commit message: Under routing
Parts:
- added C?: C_Small, symbol Device:C_Small
Connections:
- wire segments 36 -> 38
Other:
- moved on the sheet: J1, LED1, Q1, R1, R2, R3, T1, U1
